File: FLW_EkGk_Handlöten_PCB1.kicad_sch (KiCad schematic)
At the start: 1 part, among them U2 RPi-Pico

Commit message: improved
Connections:
- net LED_BUS_DIN: now reaches U2.11 (GPIO8)
- net GND: now reaches U2.13 (GND)
- net GND: now also U2.18 (GND), U2.23 (GND), U2.28 (GND), U2.3 (GND), U2.33 (AGND), U2.38 (GND), U2.42 (GND), U2.8 (GND)
- net LEDB1: no longer names the net of U2.24 (GPIO18)
- net LEDB2: no longer names the net of U2.27 (GPIO21)
- net LEDG1: no longer names the net of U2.22 (GPIO17)
- net LEDG2: no longer names the net of U2.26 (GPIO20)
- net LEDR1: no longer names the net of U2.21 (GPIO16)
- net LEDR2: no longer names the net of U2.25 (GPIO19)
Other:
- sheet Praxis 2 ports: added LED_BUS_DIN, VDD_5V; removed LED_B1, LED_B2, LED_G1, LED_G2, LED_R1, LED_R2
Changed lines of the file:
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@@
 (kicad_sch (version 20230121) (generator eeschema)
   (paper "A4")
+  (junction (at 110.49 100.33) (diameter 0) (color 0 0 0 0)
+  )
+  (junction (at 110.49 107.95) (diameter 0) (color 0 0 0 0)
+  )
+  (junction (at 110.49 97.79) (diameter 0) (color 0 0 0 0)
+  )
+  (junction (at 110.49 95.25) (diameter 0) (color 0 0 0 0)
+  )
+  (junction (at 110.49 105.41) (diameter 0) (color 0 0 0 0)
+  )
+  (junction (at 110.49 102.87) (diameter 0) (color 0 0 0 0)
+  )
+  (junction (at 110.49 119.38) (diameter 0) (color 0 0 0 0)
+  )
+  (junction (at 110.49 92.71) (diameter 0) (color 0 0 0 0)
+  )
+  (wire (pts (xy 156.845 116.84) (xy 172.72 116.84))
+    (stroke (width 0) (type default))
+  )
   (wire (pts (xy 138.43 53.34) (xy 144.78 53.34))
     (stroke (width 0) (type default))
   )
+  (wire (pts (xy 110.49 102.87) (xy 110.49 105.41))
+    (stroke (width 0) (type default))
+  )
   (wire (pts (xy 165.1 91.44) (xy 172.72 91.44))
     (stroke (width 0) (type default))
@@
     (stroke (width 0) (type default))
   )
+  (wire (pts (xy 110.49 95.25) (xy 110.49 97.79))
+    (stroke (width 0) (type default))
+  )
   (wire (pts (xy 138.43 48.26) (xy 144.78 48.26))
     (stroke (width 0) (type default))
   )
-  (wire (pts (xy 168.91 55.88) (xy 166.37 55.88))
+  (wire (pts (xy 110.49 97.79) (xy 110.49 100.33))
     (stroke (width 0) (type default))
   )
@@
     (stroke (width 0) (type default))
   )
-  (wire (pts (xy 168.91 50.8) (xy 166.37 50.8))
+  (wire (pts (xy 110.49 92.71) (xy 110.49 95.25))
     (stroke (width 0) (type default))
   )
@@
     (stroke (width 0) (type default))
   )
-  (wire (pts (xy 168.91 48.26) (xy 166.37 48.26))
-    (stroke (width 0) (type default))
-  )
   (wire (pts (xy 165.1 96.52) (xy 172.72 96.52))
     (stroke (width 0) (type default))
   )
-  (wire (pts (xy 168.91 43.18) (xy 166.37 43.18))
-    (stroke (width 0) (type default))
-  )
-  (wire (pts (xy 168.91 45.72) (xy 166.37 45.72))
+  (wire (pts (xy 110.49 90.17) (xy 110.49 92.71))
+    (stroke (width 0) (type default))
+  )
+  (wire (pts (xy 110.49 100.33) (xy 110.49 102.87))
     (stroke (width 0) (type default))
   )
@@
     (stroke (width 0) (type default))
   )
-  (wire (pts (xy 168.91 53.34) (xy 166.37 53.34))
+  (wire (pts (xy 166.37 43.18) (xy 182.245 43.18))
+    (stroke (width 0) (type default))
+  )
+  (wire (pts (xy 110.49 107.95) (xy 110.49 119.38))
+    (stroke (width 0) (type default))
+  )
+  (wire (pts (xy 110.49 105.41) (xy 110.49 107.95))
     (stroke (width 0) (type default))
   )
@@
     (effects (font (size 1.27 1.27)) (justify left bottom))
   )
-  (label "LEDR1" (at 168.91 43.18 0) (fields_autoplaced)
-    (effects (font (size 1.27 1.27)) (justify left bottom))
-  )
-  (label "LEDG1" (at 204.47 93.98 0) (fields_autoplaced)
-    (effects (font (size 1.27 1.27)) (justify left bottom))
-  )
   (label "LED2" (at 138.43 45.72 0) (fields_autoplaced)
     (effects (font (size 1.27 1.27)) (justify left bottom))
   )
-  (label "LEDB2" (at 168.91 55.88 0) (fields_autoplaced)
-    (effects (font (size 1.27 1.27)) (justify left bottom))
-  )
   (label "LED4" (at 165.1 99.06 0) (fields_autoplaced)
     (effects (font (size 1.27 1.27)) (justify left bottom))
   )
-  (label "LEDR1" (at 204.47 91.44 0) (fields_autoplaced)
-    (effects (font (size 1.27 1.27)) (justify left bottom))
-  )
   (label "LED5" (at 165.1 101.6 0) (fields_autoplaced)
     (effects (font (size 1.27 1.27)) (justify left bottom))
@@
     (effects (font (size 1.27 1.27)) (justify left bottom))
   )
-  (label "LEDG1" (at 168.91 45.72 0) (fields_autoplaced)
-    (effects (font (size 1.27 1.27)) (justify left bottom))
-  )
   (label "LED3" (at 165.1 96.52 0) (fields_autoplaced)
     (effects (font (size 1.27 1.27)) (justify left bottom))
   )
-  (label "LEDR2" (at 168.91 50.8 0) (fields_autoplaced)
-    (effects (font (size 1.27 1.27)) (justify left bottom))
-  )
-  (label "LEDG2" (at 168.91 53.34 0) (fields_autoplaced)
+  (label "LED_BUS_DIN" (at 168.91 43.18 0) (fields_autoplaced)
     (effects (font (size 1.27 1.27)) (justify left bottom))
   )
@@
     (effects (font (size 1.27 1.27)) (justify left bottom))
   )
-  (label "LEDB1" (at 168.91 48.26 0) (fields_autoplaced)
-    (effects (font (size 1.27 1.27)) (justify left bottom))
-  )
-  (label "LEDB1" (at 204.47 96.52 0) (fields_autoplaced)
-    (effects (font (size 1.27 1.27)) (justify left bottom))
-  )
   (label "LED4" (at 138.43 50.8 0) (fields_autoplaced)
     (effects (font (size 1.27 1.27)) (justify left bottom))
@@
     (effects (font (size 1.27 1.27)) (justify left bottom))
   )
-  (label "LEDB2" (at 204.47 104.14 0) (fields_autoplaced)
-    (effects (font (size 1.27 1.27)) (justify left bottom))
-  )
-  (label "LEDR2" (at 204.47 99.06 0) (fields_autoplaced)
+  (label "LED_BUS_DIN" (at 156.845 116.84 0) (fields_autoplaced)
     (effects (font (size 1.27 1.27)) (justify left bottom))
   )
@@
     (effects (font (size 1.27 1.27)) (justify left bottom))
   )
-  (label "LEDG2" (at 204.47 101.6 0) (fields_autoplaced)
-    (effects (font (size 1.27 1.27)) (justify left bottom))
-  )
   (label "LED3" (at 138.43 48.26 0) (fields_autoplaced)
     (effects (font (size 1.27 1.27)) (justify left bottom))
+  )
+  (symbol (lib_id "power:GND") (at 110.49 119.38 0) (unit 1)
+    (in_bom yes) (on_board yes) (dnp no) (fields_autoplaced)
+    (property "Reference" "#PWR060" (at 110.49 125.73 0)
+      (effects (font (size 1.27 1.27)) hide)
+    )
+    (property "Value" "GND" (at 110.49 124.46 0)
+      (effects (font (size 1.27 1.27)))
+    )
+    (property "Footprint" "" (at 110.49 119.38 0)
+      (effects (font (size 1.27 1.27)) hide)
+    )
+    (property "Datasheet" "" (at 110.49 119.38 0)
+      (effects (font (size 1.27 1.27)) hide)
+    )
+    (pin "1")
+    (instances
+      (project "FLW_EkGk_Handlöten_PCB1"
+        (path "/db211800-561f-4a5f-a2c7-7ea3433d307f/5ad671c8-fb5f-4673-842f-e2f81bf862ac"
+          (reference "#PWR060") (unit 1)
+        )
+        (path "/db211800-561f-4a5f-a2c7-7ea3433d307f"
+          (reference "#PWR067") (unit 1)
+        )
+      )
+    )
   )
   (symbol (lib_id "FabLabWintiLibrary:RPi-Pico") (at 172.72 86.36 0) (unit 1)
@@
       (effects (font (size 1.27 1.27)) (justify left))
     )
-    (pin "LED_R2" input (at 166.37 50.8 0)
+    (pin "VDD_5V" input (at 144.78 59.055 180)
+      (effects (font (size 1.27 1.27)) (justify left))
+    )
+    (pin "LED_BUS_DIN" input (at 166.37 43.18 0)
       (effects (font (size 1.27 1.27)) (justify right))
     )
-    (pin "LED_B1" input (at 166.37 48.26 0)
-      (effects (font (size 1.27 1.27)) (justify right))
-    )
-    (pin "LED_G2" input (at 166.37 53.34 0)
-      (effects (font (size 1.27 1.27)) (justify right))
-    )
-    (pin "LED_G1" input (at 166.37 45.72 0)
-      (effects (font (size 1.27 1.27)) (justify right))
-    )
-    (pin "LED_R1" input (at 166.37 43.18 0)
-      (effects (font (size 1.27 1.27)) (justify right))
-    )
-    (pin "LED_B2" input (at 166.37 55.88 0)
-      (effects (font (size 1.27 1.27)) (justify right))
-    )

Commit message: continued
Connections:
- net data: now reaches U2.21 (GPIO16)
- net clk: now reaches U2.22 (GPIO17)
- net strobe: now reaches U2.24 (GPIO18)
- net en: now reaches U2.25 (GPIO19)
- net +5V: now reaches U2.40 (VBUS)
- net LED1 renamed led1
- net LED2 renamed led2
- net LED3 renamed led3
- net LED4 renamed led4
- net LED5 renamed led5
- net LED6 renamed led6
- net LED_BUS_DIN renamed led_bus_din
Other:
- sheet Praxis 3 ports: added +5V0, CLK, DATA, EN, STROBE; removed none
- moved on the sheet: U2A, U2B

Commit message: Almost finished
Connections:
- net +3V3: now reaches U2.36 (3V3)
- no-connect marks 0 -> 20
Other:
- sheet Praxis 3 ports: added +3V3; removed none
- moved on the sheet: U2A, U2B
