File: FLW_EkGk_Handlöten_PCB1.kicad_sch (KiCad schematic)
At the start: 1 part, among them U2 RPi-Pico

Commit message: resolved RGB issue
Connections:
- no-connect marks 20 -> 21
Changed lines of the file:
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@@
+	)
+	(no_connect
+		(at 118.11 124.46)
 	)
 	(no_connect
