File: Praxis2.kicad_sch (KiCad schematic)
At the start: 18 parts, among them Q60 2N7002, Q61 2N7002, Q62 2N7002, Q63 2N7002, Q64 2N7002, Q65 2N7002

Commit message: continued
Parts:
- added LED66, LED67: SMLP36RGBNW3, NiksKiCadLibrary:LED_SMLP36_ROM, symbol NiksKiCadLibrary:SMLP36RGBNW3
- added R21 (x6): R, Resistor_SMD:R_1206_3216Metric, symbol Device:R
Connections:
- net GND: now also LED66.4, LED66.5, LED66.6, LED67.4, LED67.5, LED67.6
- net LED_B1: now also R21.1
- net LED_B2: now also R21.1
- net LED_G1: now also R21.1
- net LED_G2: now also R21.1
- net LED_R1: now also R21.1
- net LED_R2: now also R21.1
- net VDD_5V: now reaches R21.1
- net VDD_5V: now also R21.1, R21.1, R21.1, R21.1, R21.1
- new net: LED67.1, R21.2
- new net: LED67.2, R21.2
- new net: LED67.3, R21.2
- new net: LED66.1, R21.2
- new net: LED66.3, R21.2
- new net: LED66.2, R21.2

Commit message: improved
Parts:
- removed LED66, LED67: SMLP36RGBNW3, NiksKiCadLibrary:LED_SMLP36_ROM, symbol NiksKiCadLibrary:SMLP36RGBNW3
- removed R21 (x6): R, Resistor_SMD:R_1206_3216Metric, symbol Device:R
- added LED66, LED67, LED68: LTST-E563CEGBW, NiksKiCadLibrary:LTSTE563CEGBW, symbol NiksKiCadLibrary:LTST-E563CEGBW
Connections:
- net GND: now also LED66.1 (VSS), LED67.1 (VSS), LED68.1 (VSS)
- net VDD_5V: now also LED66.4 (VDD), LED67.4 (VDD), LED68.4 (VDD)
- new net: LED66.3 (DOUT), LED67.2 (DIN)
- new net: LED67.3 (DOUT), LED68.2 (DIN)
- new net LED_BUS_DIN: LED66.2 (DIN)
Other:
- moved on the sheet: LED60, LED61, LED62, LED63, LED64, LED65, Q60, Q61, Q62, Q63, Q64, Q65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

Commit message: Resolves #2: Added current limiting resistor values (i.e. 620 Ohm)
Parts:
- R60, R61, R62, R63, R64, R65: renamed from R21; value R -> 620R
