File: Praxis2.kicad_sch (KiCad schematic)
At the start: 21 parts, among them Q60 2N7002, Q61 2N7002, Q62 2N7002, Q63 2N7002, Q64 2N7002, Q65 2N7002

Commit message: resolved RGB issue
Parts:
- added Q73: 2N7002, Package_TO_SOT_SMD:SOT-23, symbol Transistor_FET:2N7002
- added R79: 10k, Resistor_SMD:R_1206_3216Metric, symbol Device:R
Connections:
- net GND: now also Q73.2 (S)
- net LED_BUS_DIN: now also Q73.1 (G); no longer LED66.2 (DIN)
- net VDD_5V: now also R79.1
- new net: LED66.2 (DIN), Q73.3 (D), R79.2
Other:
- moved on the sheet: LED66, LED67, LED68
