File: Praxis1.kicad_sch (KiCad schematic)
At the start: 44 parts, among them J10 Conn_01x02, J11 Conn_01x02, J12 Conn_01x02, J13 Conn_01x02

Commit message: asdf
Parts:
- removed J10, J11, J12, J13: Conn_01x02, Connector_PinHeader_2.54mm:PinHeader_1x02_P2.54mm_Horizontal, symbol Connector_Generic:Conn_01x02
- removed R37: R, Resistor_SMD:R_1206_3216Metric, symbol Device:R
- removed R47: R, Resistor_SMD:R_0805_2012Metric, symbol Device:R
Connections:
- net at R40.1, R41.1, R42.1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: no longer R48.1, R49.1
- net at R40.2, R41.2, R42.2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: no longer R48.2, R49.2
- net at R38.1: now also R39.1
- net GND: now reaches R38.2, R39.2
- net GND: now also R48.2, R49.2
- net at R19.1: now also R10.1
- net at R30.1: now also R36.2
- new net: R48.1, R49.1
Other:
- note added: "Komponenten mit starker Wärmeleitkopplung"
- moved on the sheet: R10, R11, R12, R13, R14, R15, R16, R17, R18, R19, R20, R21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
