File: Praxis3.kicad_sch (KiCad schematic)
At the start: 48 parts, among them IC60 HCF4094YM013TR, IC61 HCF4094YM013TR, Q66 2N7002, Q67 2N7002, Q68 2N7002, Q69 2N7002, Q70 2N7002, Q71 2N7002, Q72 2N7002, SW60 MSS6-V-T_R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

Commit message: asdf
Parts:
- removed SW61, SW62: B3U-3100P, SW_B3U-3100P_OMR, symbol NiksKiCadLibrary:B3U-3100P
- added SW63, SW64: SW_Push, Button_Switch_SMD:SW_Push_1P1T_NO_CK_KSC7xxJ, symbol Switch:SW_Push
Connections:
- net GND: now also SW63.2, SW64.2
- net at R74.1: now also SW63.1
- net at R66.1: now also SW64.1
