File: FLW_EkGk_Handlöten_PCB1.kicad_pcb (KiCad board)
At the start: 2 copper layers, 120 x 66 mm, 110 parts, among them IC60 HCF4094YM013TR, IC61 HCF4094YM013TR, Q60 2N7002, Q61 2N7002, Q62 2N7002, Q63 2N7002, Q64 2N7002, Q65 2N7002, Q66 2N7002, Q67 2N7002, Q68 2N7002, Q69 2N7002, Q70 2N7002, Q71 2N7002, Q72 2N7002, SW60 MSS6-V-T_R, SW61 B3U-3100P, SW62 B3U-3100P, U2 RPi-Pico

Commit message: resolved RGB issue
Parts:
- removed SW61, SW62: B3U-3100P, NiksKiCadLibrary:SW_B3U-3100P_OMR
- added Q73: 2N7002, Package_TO_SOT_SMD:SOT-23, F.Cu at (155.0, 69.5)
- added R79: 10k, Resistor_SMD:R_1206_3216Metric, F.Cu at (154.5, 64.0)
- added SW63: SW_Push, Button_Switch_SMD:SW_Push_1P1T_NO_CK_KSC7xxJ, F.Cu at (96.5, 84.5)
- added SW64: SW_Push, Button_Switch_SMD:SW_Push_1P1T_NO_CK_KSC7xxJ, F.Cu at (96.5, 103.0)
- moved R74 11.9 mm to (104.5, 100.0), turned to -90 degrees
- moved R66 10.8 mm to (104.5, 105.5), turned to -90 degrees
- moved SW60 8.64 mm to (96.8, 93.8)
- moved C64 2.93 mm to (110.5, 101.3)
- moved C66 2.93 mm to (116.2, 101.3)
- moved R76 2.93 mm to (110.5, 106.4)
- moved R77 2.93 mm to (113.4, 106.4)
- moved R78 2.93 mm to (116.2, 106.4)
- moved C63 2.93 mm to (107.6, 101.3)
- moved C65 2.93 mm to (113.4, 101.3)
- moved R75 2.93 mm to (107.6, 106.4)
- moved LED66 2.10 mm to (160.0, 63.8)
- moved LED67 2.10 mm to (165.4, 54.5)
- moved LED68 2.10 mm to (171.0, 63.8)
Connections:
- LED66 pad 2: /led_bus_din -> Net-(LED66-DIN)
- R38 pad 1: Net-(R38-Pad1) -> GND
- R39 pad 1: Net-(R38-Pad1) -> GND
- R48 pad 1: Net-(R48-Pad1) -> GND
- R49 pad 1: Net-(R48-Pad1) -> GND
Routing:
- net Net-(R74-Pad1): track 8.36 -> 30.1 mm
- net /clk: track 87.2 -> 74.4 mm
- net /Praxis 3/+3v3: track 20.3 -> 32.9 mm, vias 0 -> 2
- net Net-(LED66-DIN): track 0.00 -> 11.9 mm
- net /Praxis 3/+5v0: track 128.1 -> 117.4 mm
- net /+3V3: track 114.1 -> 123.9 mm, vias 0 -> 2
- net /data: track 76.5 -> 68.0 mm
- net /led_bus_din: track 42.4 -> 34.5 mm
- net /+5V: track 240.1 -> 233.0 mm, vias 2 -> 0
- net Net-(R48-Pad1): track 6.00 -> 0.00 mm
- net Net-(R38-Pad1): track 6.00 -> 0.00 mm
- net Net-(R66-Pad1): track 7.38 -> 11.3 mm
- net /en: track 75.8 -> 73.0 mm
- net /strobe: track 69.9 -> 67.9 mm
- net /Praxis 3/led1: track 16.2 -> 17.8 mm
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Other:
- board text added: "16. August 2026 - Release 2.0"
- board text added: "HCF4094"
- board text removed: "13. Mai 2026 - Release 1.4"
